File: wemos hat.sch (KiCad schematic (older format))
At the start: 16 parts, among them J1 RJ45, U1 MAX3072E, U2 WeMos_mini

Commit message: Components done
Parts:
- R1, R2, R3, R4, R5, R6: footprint Resistor_SMD:R_0402_1005Metric -> Resistor_SMD:R_0603_1608Metric
- renumbered BUCK?1 to BUCK1
Changed lines of the file:
@@
 $EndDescr
 $Comp
-L MyLib:MP1584 BUCK?1
+L MyLib:MP1584 BUCK1
 U 1 1 5DEBF823
 P 3750 5400
-F 0 "BUCK?1" H 3750 5775 50  0000 C CNN
+F 0 "BUCK1" H 3750 5775 50  0000 C CNN
 F 1 "MP1584" H 3750 5684 50  0000 C CNN
 F 2 "Package_SO:SOIC-8_3.9x4.9mm_P1.27mm" H 3650 5300 50  0001 C CNN
@@
 F 0 "R2" V 3057 5250 50  0000 C CNN
 F 1 "100k" V 2966 5250 50  0000 C CNN
-F 2 "Resistor_SMD:R_0402_1005Metric" V 2780 5250 50  0001 C CNN
+F 2 "Resistor_SMD:R_0603_1608Metric" V 2780 5250 50  0001 C CNN
 F 3 "~" H 2850 5250 50  0001 C CNN
 	1    2850 5250
@@
 F 0 "R3" H 3120 5646 50  0000 L CNN
 F 1 "200k" H 3120 5555 50  0000 L CNN
-F 2 "Resistor_SMD:R_0402_1005Metric" V 2980 5600 50  0001 C CNN
+F 2 "Resistor_SMD:R_0603_1608Metric" V 2980 5600 50  0001 C CNN
 F 3 "~" H 3050 5600 50  0001 C CNN
 	1    3050 5600
@@
 F 0 "R1" H 2770 5546 50  0000 L CNN
 F 1 "24.9k" H 2770 5455 50  0000 L CNN
-F 2 "Resistor_SMD:R_0402_1005Metric" V 2630 5500 50  0001 C CNN
+F 2 "Resistor_SMD:R_0603_1608Metric" V 2630 5500 50  0001 C CNN
 F 3 "~" H 2700 5500 50  0001 C CNN
 	1    2700 5500
@@
 F 0 "R4" H 4170 6046 50  0000 L CNN
 F 1 "68.1k" H 4170 5955 50  0000 L CNN
-F 2 "Resistor_SMD:R_0402_1005Metric" V 4030 6000 50  0001 C CNN
+F 2 "Resistor_SMD:R_0603_1608Metric" V 4030 6000 50  0001 C CNN
 F 3 "~" H 4100 6000 50  0001 C CNN
 	1    4100 6000
@@
 F 0 "R5" H 5020 5646 50  0000 L CNN
 F 1 "40.2k" H 5020 5555 50  0000 L CNN
-F 2 "Resistor_SMD:R_0402_1005Metric" V 4880 5600 50  0001 C CNN
+F 2 "Resistor_SMD:R_0603_1608Metric" V 4880 5600 50  0001 C CNN
 F 3 "~" H 4950 5600 50  0001 C CNN
 	1    4950 5600
@@
 F 0 "R6" V 5043 5450 50  0000 C CNN
 F 1 "124k" V 5134 5450 50  0000 C CNN
-F 2 "Resistor_SMD:R_0402_1005Metric" V 5180 5450 50  0001 C CNN
+F 2 "Resistor_SMD:R_0603_1608Metric" V 5180 5450 50  0001 C CNN
 F 3 "~" H 5250 5450 50  0001 C CNN
 	1    5250 5450
